Commit message: Initial paro work

File: sensors/paro.xacro (robot description, xacro)
@@ -3,5 +3,5 @@
 <xacro:macro name="paro_digiquartz" params="name parent_link xyz rpy">
   <!-- First, define the link -->
-  <link name="${name}">
+  <link name="${name}_link">
     <visual>
       <origin xyz="0 0 0.1217" rpy="0 0 0"/>
@@ -12,11 +12,30 @@
     </visual>
   </link>
+    <gazebo reference="${parent_link}">
+      <sensor name="${name}_sensor" type="dsros_depth">
+        <always_on>1</always_on>
+        <update_rate>5.000</update_rate>
+        <pose frame="">${xyz} ${rpy}</pose>
+        <dsros_depth>
+        </dsros_depth>
+      </sensor>
+    </gazebo>
   <!-- Now apply the offsets -->
   <joint name="base_to_${name}" type="fixed">
     <parent link="${parent_link}"/>
-    <child link="${name}"/>
+    <child link="${name}_link"/>
     <origin xyz="${xyz}" rpy="${rpy}"/>
   </joint>
-  <!-- TODO: Gazebo plugin to actually take measurements! -->
+  <!-- Gazebo plugin to actually take measurements! -->
+  <gazebo>
+    <!--
+    <plugin name="depthsensor_${name}" filename="libdsros_depthsensor.so">
+      <robotNamespace>$(arg namespace)</robotNamespace>
+      <root_topic>sensors/${name}</root_topic>
+      <linkname>${name}</linkname>
+      <updateRate>5</updateRate>
+    </plugin>
+    -->
+  </gazebo>
 </xacro:macro>
 </robot>

Commit message: Initial sensor commit.  Working depth!

File: sensors/paro.xacro (robot description, xacro)
@@ -1,5 +1,5 @@
 <?xml version="1.0"?>
 <robot xmlns:xacro="http://www.ros.org/wiki/xacro">
-<xacro:macro name="paro_digiquartz" params="name parent_link xyz rpy">
+<xacro:macro name="paro_digiquartz" params="name parent_link xyz rpy robot_namespace topic">
   <!-- First, define the link -->
   <link name="${name}_link">
@@ -12,13 +12,22 @@
     </visual>
   </link>
-    <gazebo reference="${parent_link}">
-      <sensor name="${name}_sensor" type="dsros_depth">
-        <always_on>1</always_on>
-        <update_rate>5.000</update_rate>
-        <pose frame="">${xyz} ${rpy}</pose>
-        <dsros_depth>
-        </dsros_depth>
-      </sensor>
-    </gazebo>
+  <gazebo reference="${name}_link">
+    <material>Gazebo/Grey</material>
+  </gazebo>
+  <gazebo reference="${parent_link}">
+    <sensor name="${name}_sensor" type="dsros_depth">
+      <always_on>1</always_on>
+      <update_rate>5.000</update_rate>
+      <pose frame="">${xyz} ${rpy}</pose>
+      <plugin name="${name}_sensor_controller" filename="libdsros_ros_depth.so">
+          <robotNamespace>${robot_namespace}</robotNamespace>
+          <topicName>${topic}</topicName>
+          <frameName>world</frameName>
+          <updateRateHZ>5</updateRateHZ>
+          <!-- Actually in decibars, but pretty close to meters -->
+          <gaussianNoise>0.005</gaussianNoise>
+      </plugin>
+    </sensor>
+  </gazebo>
   <!-- Now apply the offsets -->
   <joint name="base_to_${name}" type="fixed">
@@ -27,15 +36,4 @@
     <origin xyz="${xyz}" rpy="${rpy}"/>
   </joint>
-  <!-- Gazebo plugin to actually take measurements! -->
-  <gazebo>
-    <!--
-    <plugin name="depthsensor_${name}" filename="libdsros_depthsensor.so">
-      <robotNamespace>$(arg namespace)</robotNamespace>
-      <root_topic>sensors/${name}</root_topic>
-      <linkname>${name}</linkname>
-      <updateRate>5</updateRate>
-    </plugin>
-    -->
-  </gazebo>
 </xacro:macro>
 </robot>

File: sensors/phins.xacro (robot description, xacro)
@@ -1,6 +1,6 @@
 <?xml version="1.0"?>
 <robot xmlns:xacro="http://www.ros.org/wiki/xacro">
-<xacro:macro name="phins" params="name parent_link xyz rpy">
-  <link name="phins">
+<xacro:macro name="phins" params="name parent_link xyz rpy robot_namespace ins_topic att_topic">
+  <link name="${name}_link">
     <visual>
       <origin xyz="0.0082 -0.0043 -0.0066" rpy="0 0 0"/>
@@ -11,7 +11,26 @@
     </visual>
   </link>
+  <gazebo reference="${name}_link">
+    <material>Gazebo/Grey</material>
+  </gazebo>
+  <gazebo reference="${parent_link}">
+    <sensor name="${name}_sensor" type="dsros_ins">
+      <always_on>1</always_on>
+      <update_rate>10.000</update_rate>
+      <pose frame="">${xyz} ${rpy}</pose>
+      <plugin name="${name}_sensor_controller" filename="libdsros_ros_ins.so">
+        <robotNamespace>${robot_namespace}</robotNamespace>
+        <insTopicName>${ins_topic}</insTopicName>
+        <attTopicName>${att_topic}</attTopicName>
+        <frameName>world</frameName>
+        <updateRateHZ>10</updateRateHZ>
+        <gaussianNoisePR>0.001</gaussianNoisePR>
+        <gaussianNoiseY>0.01</gaussianNoiseY>
+      </plugin>
+    </sensor>
+  </gazebo>
   <joint name="base_to_phins" type="fixed">
     <parent link="${parent_link}"/>
-    <child link="phins"/>
+    <child link="${name}_link"/>
     <origin xyz="${xyz}" rpy="${rpy}"/>
   </joint>
