Commit message: Fixed assorted gps_plugin issues.  Works now

File: sensors/xeos_gps.xacro (robot description, xacro)
@@ -1,5 +1,5 @@
 <?xml version="1.0"?>
 <robot xmlns:xacro="http://www.ros.org/wiki/xacro">
-<xacro:macro name="xeos_gps" params="name parent_link xyz rpy">
+<xacro:macro name="xeos_gps" params="name parent_link xyz rpy robot_namespace topic">
   <!-- First, define the link -->
   <link name="${name}">
@@ -18,5 +18,22 @@
     <origin xyz="${xyz}" rpy="${rpy}"/>
   </joint>
-  <!-- TODO: Gazebo plugin to actually take measurements! -->
+  <!-- Gazebo plugin to actually take measurements! -->
+  <gazebo reference="${parent_link}">
+    <sensor name="${name}_sensor" type="gps">
+      <always_on>1</always_on>
+      <update_rate>1.0</update_rate>
+      <pose frame="">${xyz} ${rpy}</pose>
+      <plugin name="${name}_sensor_controller" filename="libdsros_ros_gps.so">
+        <robotNamespace>${robot_namespace}</robotNamespace>
+        <topicName>${topic}</topicName>
+        <frameName>world</frameName>
+        <updateRateHZ>1.0</updateRateHZ>
+        <!-- Minimum altitude (- max depth) at which we get a position fix -->
+        <minAltitude>0.01</minAltitude>
+        <gaussianNoiseLL_meters>1.0</gaussianNoiseLL_meters>
+        <gaussianNoiseAlt_meters>2.0</gaussianNoiseAlt_meters>
+      </plugin>
+    </sensor>
+  </gazebo>
 </xacro:macro>
 </robot>
