Commit message: Staging for the split between runtime and sim xacro

File: sensors/avtrak.xacro (robot description, xacro)
@@ -1,5 +1,5 @@
 <?xml version="1.0"?>
 <robot xmlns:xacro="http://www.ros.org/wiki/xacro">
-<xacro:macro name="avtrak" params="name parent_link xyz rpy">
+<xacro:macro name="avtrak" params="name parent_link xyz rpy **sim">
   <!-- First, define the link -->
   <link name="${name}">
@@ -18,5 +18,6 @@
     <origin xyz="${xyz}" rpy="${rpy}"/>
   </joint>
-  <!-- TODO: Gazebo plugin to actually take measurements! -->
+  <!-- Gazebo stuff for Avtrak, if applicable -->
+  <xacro:insert_block name="sim"/>
 </xacro:macro>
 </robot>

File: sensors/paro.xacro (robot description, xacro)
@@ -1,5 +1,5 @@
 <?xml version="1.0"?>
 <robot xmlns:xacro="http://www.ros.org/wiki/xacro">
-<xacro:macro name="paro_digiquartz" params="name parent_link xyz rpy robot_namespace topic">
+<xacro:macro name="paro_digiquartz" params="name parent_link xyz rpy **sim">
   <!-- First, define the link -->
   <link name="${name}_link">
@@ -12,23 +12,5 @@
     </visual>
   </link>
-  <gazebo reference="${name}_link">
-    <material>Gazebo/Grey</material>
-  </gazebo>
-  <gazebo reference="${parent_link}">
-    <sensor name="${name}_sensor" type="dsros_depth">
-      <always_on>1</always_on>
-      <update_rate>5.000</update_rate>
-      <pose frame="">${xyz} ${rpy}</pose>
-      <plugin name="${name}_sensor_controller" filename="libdsros_ros_depth.so">
-          <robotNamespace>${robot_namespace}</robotNamespace>
-          <topicName>${topic}</topicName>
-          <frameName>world</frameName>
-          <updateRateHZ>5</updateRateHZ>
-          <!-- Actually in decibars, but pretty close to meters -->
-          <gaussianNoise>0.005</gaussianNoise>
-      </plugin>
-    </sensor>
-  </gazebo>
-  <!-- Now apply the offsets -->
+   <!-- Now apply the offsets -->
   <joint name="base_to_${name}" type="fixed">
     <parent link="${parent_link}"/>
@@ -36,4 +18,6 @@
     <origin xyz="${xyz}" rpy="${rpy}"/>
   </joint>
+  <!-- Gazebo sim stuff, if applicable -->
+  <xacro:insert_block name="sim"/>
 </xacro:macro>
 </robot>

File: sensors/phins.xacro (robot description, xacro)
@@ -1,5 +1,5 @@
 <?xml version="1.0"?>
 <robot xmlns:xacro="http://www.ros.org/wiki/xacro">
-<xacro:macro name="phins" params="name parent_link xyz rpy robot_namespace ins_topic att_topic">
+<xacro:macro name="phins" params="name parent_link xyz rpy **sim">
   <link name="${name}_link">
     <visual>
@@ -11,27 +11,4 @@
     </visual>
   </link>
-  <gazebo reference="${name}_link">
-    <material>Gazebo/Grey</material>
-  </gazebo>
-  <gazebo reference="${parent_link}">
-    <sensor name="${name}_sensor" type="dsros_ins">
-      <always_on>1</always_on>
-      <update_rate>10.000</update_rate>
-      <pose frame="">${xyz} ${rpy}</pose>
-      <plugin name="${name}_sensor_controller" filename="libdsros_ros_ins.so">
-        <robotNamespace>${robot_namespace}</robotNamespace>
-        <insTopicName>${ins_topic}</insTopicName>
-        <attTopicName>${att_topic}</attTopicName>
-        <frameName>world</frameName>
-        <updateRateHZ>10</updateRateHZ>
-        <gaussianNoisePR>0.001</gaussianNoisePR>
-        <gaussianNoiseY>0.01</gaussianNoiseY>
-        <gaussianNoiseVel>0.01</gaussianNoiseVel>
-        <gaussianNoiseAngVel>0.01</gaussianNoiseAngVel>
-        <gaussianNoiseAcc>0.01</gaussianNoiseAcc>
-        <gaussianNoiseLat>0.1</gaussianNoiseLat>
-      </plugin>
-    </sensor>
-  </gazebo>
   <joint name="base_to_phins" type="fixed">
     <parent link="${parent_link}"/>
@@ -39,4 +16,6 @@
     <origin xyz="${xyz}" rpy="${rpy}"/>
   </joint>
+  <!-- Gazebo sim stuff, if applicable -->
+  <xacro:insert_block name="sim"/>
 </xacro:macro>
 </robot>

File: sensors/rdi300.xacro (robot description, xacro)
@@ -1,5 +1,5 @@
 <?xml version="1.0"?>
 <robot xmlns:xacro="http://www.ros.org/wiki/xacro">
-<xacro:macro name="rdi_workhorse_300" params="name parent_link xyz rpy robot_namespace dvl_topic">
+<xacro:macro name="rdi_workhorse_300" params="name parent_link xyz rpy **sim">
   <!-- First, define the link -->
   <link name="${name}">
@@ -12,33 +12,4 @@
     </visual>
   </link>
-  <gazebo reference="${name}_link">
-    <material>Gazebo/Green</material>
-  </gazebo>
-  <gazebo reference="${parent_link}">
-    <sensor name="${name}_sensor" type="dsros_dvl">
-      <always_on>1</always_on>
-      <update_rate>2.0</update_rate>
-      <pose frame="">${xyz} ${rpy}</pose>
-      <!-- doesn't do anything atm.  Bummer.
-      <dvl>
-        300kHz DVL
-        <minRange>1.0</minRange>
-        <maxRange>200</maxRange>
-        <maxRangeDiff>10</maxRangeDiff>
-        <beamAngleDeg>30.0</beamAngleDeg>
-        <beamWidthDeg>4.0</beamWidthDeg>
-      </dvl>
-      -->
-      <plugin name="${name}_sensor_controller" filename="libdsros_ros_dvl.so">
-        <robotNamespace>${robot_namespace}</robotNamespace>
-        <topicName>${dvl_topic}</topicName>
-        <frameName>${name}</frameName>
-        <pointcloudFrame>${parent_link}</pointcloudFrame>
-        <updateRateHZ>2.0</updateRateHZ>
-        <gaussianNoiseBeamVel>0.01</gaussianNoiseBeamVel>
-        <gaussianNoiseBeamRange>0.1</gaussianNoiseBeamRange>
-      </plugin>
-    </sensor>
-  </gazebo>
   <!-- Now apply the offsets -->
   <joint name="base_to_${name}" type="fixed">
@@ -47,20 +18,6 @@
     <origin xyz="${xyz}" rpy="${rpy}"/>
   </joint>
-        <!--  600kHz DVL -->
-        <!--
-        <minRange>0.7</minRange>
-        <maxRange>90</maxRange>
-        <maxRangeDiff>10</maxRangeDiff>
-        <beamAngleDeg>30.0</beamAngleDeg>
-        <beamWidthDeg>2.0</beamWidthDeg>
-        -->
-        <!-- 1200kHz DVL -->
-        <!--
-        <minRange>0.5</minRange>
-        <maxRange>45</maxRange>
-        <maxRangeDiff>10</maxRangeDiff>
-        <beamAngleDeg>30.0</beamAngleDeg>
-        <beamWidthDeg>1.5</beamWidthDeg>
-        -->
+  <!-- Gazebo sim stuff, if applicable -->
+  <xacro:insert_block name="sim"/>
 </xacro:macro>
 </robot>

File: sensors/xeos_gps.xacro (robot description, xacro)
@@ -1,5 +1,5 @@
 <?xml version="1.0"?>
 <robot xmlns:xacro="http://www.ros.org/wiki/xacro">
-<xacro:macro name="xeos_gps" params="name parent_link xyz rpy robot_namespace topic">
+<xacro:macro name="xeos_gps" params="name parent_link xyz rpy **sim">
   <!-- First, define the link -->
   <link name="${name}">
@@ -18,22 +18,6 @@
     <origin xyz="${xyz}" rpy="${rpy}"/>
   </joint>
-  <!-- Gazebo plugin to actually take measurements! -->
-  <gazebo reference="${parent_link}">
-    <sensor name="${name}_sensor" type="gps">
-      <always_on>1</always_on>
-      <update_rate>1.0</update_rate>
-      <pose frame="">${xyz} ${rpy}</pose>
-      <plugin name="${name}_sensor_controller" filename="libdsros_ros_gps.so">
-        <robotNamespace>${robot_namespace}</robotNamespace>
-        <topicName>${topic}</topicName>
-        <frameName>world</frameName>
-        <updateRateHZ>1.0</updateRateHZ>
-        <!-- Minimum altitude (- max depth) at which we get a position fix -->
-        <minAltitude>0.01</minAltitude>
-        <gaussianNoiseLL_meters>1.0</gaussianNoiseLL_meters>
-        <gaussianNoiseAlt_meters>2.0</gaussianNoiseAlt_meters>
-      </plugin>
-    </sensor>
-  </gazebo>
+  <!-- Gazebo sim stuff, if applicable -->
+  <xacro:insert_block name="sim"/>
 </xacro:macro>
 </robot>
