Commit message: Updates from nav integration

File: urdf/phins_sim.xacro (robot description, xacro)
@@ -1,5 +1,5 @@
 <?xml version="1.0"?>
 <robot xmlns:xacro="http://www.ros.org/wiki/xacro">
-<xacro:macro name="phins_sim" params="name parent_link xyz rpy robot_namespace ins_topic att_topic">
+<xacro:macro name="phins_sim" params="name parent_link xyz rpy robot_namespace ins_topic gyro_topic att_topic">
   <gazebo reference="${name}_link">
     <material>Gazebo/Grey</material>
@@ -13,4 +13,5 @@
         <robotNamespace>${robot_namespace}</robotNamespace>
         <insTopicName>${ins_topic}</insTopicName>
+        <gyroTopicName>${gyro_topic}</gyroTopicName>
         <attTopicName>${att_topic}</attTopicName>
         <frameName>world</frameName>
