Commit message: Non-flat terrain option in gazebo

File: urdf/rdi300_sim.xacro (robot description, xacro)
@@ -1,5 +1,5 @@
 <?xml version="1.0"?>
 <robot xmlns:xacro="http://www.ros.org/wiki/xacro">
-<xacro:macro name="rdi_workhorse_300_sim" params="name parent_link xyz rpy robot_namespace dvl_topic">
+<xacro:macro name="rdi_workhorse_300_sim" params="name parent_link xyz rpy robot_namespace dvl_topic ranges_topic">
   <gazebo reference="${name}_link">
     <material>Gazebo/Green</material>
@@ -23,4 +23,5 @@
         <robotNamespace>${robot_namespace}</robotNamespace>
         <topicName>${dvl_topic}</topicName>
+        <rangesTopicName>${ranges_topic}</rangesTopicName>
         <frameName>${name}_link</frameName>
         <pointcloudFrame>${parent_link}</pointcloudFrame>
