Commit message: Support for many things, including demo sonars, multiple DVL defintions, etc

File: urdf/basic_camera_sim.xacro (robot description, xacro)
@@ -25,14 +25,40 @@
 -->
 <robot xmlns:xacro="http://www.ros.org/wiki/xacro">
-<xacro:include filename="$(find ds_sim)/urdf/phins_sim.xacro"/>
-<xacro:include filename="$(find ds_sim)/urdf/paro_sim.xacro"/>
-<xacro:include filename="$(find ds_sim)/urdf/rdi300_sim.xacro"/>
-<xacro:include filename="$(find ds_sim)/urdf/nortek1000_sim.xacro"/>
-<xacro:include filename="$(find ds_sim)/urdf/xeos_gps_sim.xacro"/>
-<xacro:include filename="$(find ds_sim)/urdf/avtrak_sim.xacro"/>
-<xacro:include filename="$(find ds_sim)/urdf/resonAUV3_sim.xacro"/>
-<xacro:include filename="$(find ds_sim)/urdf/norbitWBMS_bathy_sim.xacro"/>
-<xacro:include filename="$(find ds_sim)/urdf/norbitWBMS_3D_sim.xacro"/>
-<xacro:include filename="$(find ds_sim)/urdf/basic_camera_sim.xacro"/>
-<xacro:include filename="$(find ds_sim)/urdf/dspl_seasphere_sim.xacro"/>
+<xacro:macro name="basic_camera_sim" params="name parent_link xyz rpy cam_namespace">
+  <gazebo reference="${name}_link">
+      <material>Gazebo/Red</material>
+  </gazebo>
+  <gazebo reference="${name}_link">
+    <sensor type="camera" name="${name}_sensor">
+        <update_rate>10.0</update_rate>
+        <!--<pose frame="">${xyz} ${rpy}</pose>-->
+        <camera name="${name}_camera">
+          <horizontal_fov>${pi/2}</horizontal_fov>
+          <image>
+              <width>640</width>
+              <height>480</height>
+              <format>R8G8B8</format>
+          </image>
+          <clip>
+            <near>0.02</near>
+            <far>20</far>
+          </clip>
+        </camera>
+        <plugin name="camera_controller" filename="libgazebo_ros_camera.so">
+            <alwaysOn>true</alwaysOn>
+            <updateRate>10.0</updateRate>
+            <cameraName>${cam_namespace}</cameraName>
+            <imageTopicName>image</imageTopicName>
+            <cameraInfoTopicName>camera_info</cameraInfoTopicName>
+            <frame_name>${name}_link</frame_name>
+            <hackBaseline>0.0</hackBaseline>
+            <distortionK1>0.0</distortionK1>
+            <distortionK2>0.0</distortionK2>
+            <distortionK3>0.0</distortionK3>
+            <distortionT1>0.0</distortionT1>
+            <distortionT2>0.0</distortionT2>
+        </plugin>
+    </sensor>
+  </gazebo>
+</xacro:macro>
 </robot>

File: urdf/dspl_seasphere_sim.xacro (robot description, xacro)
@@ -1,5 +1,5 @@
 <?xml version="1.0"?>
 <!--
-Copyright 2018 Woods Hole Oceanographic Institution
+Copyright 2019 Woods Hole Oceanographic Institution
 Redistribution and use in source and binary forms, with or without
 modification, are permitted provided that the following conditions are met:
@@ -25,14 +25,30 @@
 -->
 <robot xmlns:xacro="http://www.ros.org/wiki/xacro">
-<xacro:include filename="$(find ds_sim)/urdf/phins_sim.xacro"/>
-<xacro:include filename="$(find ds_sim)/urdf/paro_sim.xacro"/>
-<xacro:include filename="$(find ds_sim)/urdf/rdi300_sim.xacro"/>
-<xacro:include filename="$(find ds_sim)/urdf/nortek1000_sim.xacro"/>
-<xacro:include filename="$(find ds_sim)/urdf/xeos_gps_sim.xacro"/>
-<xacro:include filename="$(find ds_sim)/urdf/avtrak_sim.xacro"/>
-<xacro:include filename="$(find ds_sim)/urdf/resonAUV3_sim.xacro"/>
-<xacro:include filename="$(find ds_sim)/urdf/norbitWBMS_bathy_sim.xacro"/>
-<xacro:include filename="$(find ds_sim)/urdf/norbitWBMS_3D_sim.xacro"/>
-<xacro:include filename="$(find ds_sim)/urdf/basic_camera_sim.xacro"/>
-<xacro:include filename="$(find ds_sim)/urdf/dspl_seasphere_sim.xacro"/>
+<xacro:macro name="dspl_seasphere_sim" params="name parent_link xyz rpy">
+  <gazebo reference="${name}_link">
+      <material>Gazebo/Red</material>
+  </gazebo>
+  <gazebo>
+    <plugin name="${name}_light_plugin" filename="libdsros_spotlight.so">
+        <pose>${xyz} ${rpy}</pose>
+        <light type="spot" name="${name}_light">
+            <diffuse>1 1 1 1</diffuse>
+            <specular>0.1 0.1 0.1 1.0</specular>
+            <attenuation>
+                <range>20</range>
+                <linear>0.2</linear>
+                <constant>0.8</constant>
+                <quadratic>0.01</quadratic>
+            </attenuation>
+            <cast_shadows>true</cast_shadows>">
+            <direction>1 0 0</direction>
+            <spot>
+                <inner_angle>${pi/180*75}</inner_angle>
+                <outer_angle>${pi/180*115}</outer_angle>
+                <falloff>1.0</falloff>
+            </spot>
+        </light>
+    </plugin>
+  </gazebo>
+</xacro:macro>
 </robot>

File: urdf/norbitWBMS_3D_sim.xacro (robot description, xacro)
@@ -1,5 +1,5 @@
 <?xml version="1.0"?>
 <!--
-Copyright 2018 Woods Hole Oceanographic Institution
+Copyright 2019 Woods Hole Oceanographic Institution
 Redistribution and use in source and binary forms, with or without
 modification, are permitted provided that the following conditions are met:
@@ -25,14 +25,38 @@
 -->
 <robot xmlns:xacro="http://www.ros.org/wiki/xacro">
-<xacro:include filename="$(find ds_sim)/urdf/phins_sim.xacro"/>
-<xacro:include filename="$(find ds_sim)/urdf/paro_sim.xacro"/>
-<xacro:include filename="$(find ds_sim)/urdf/rdi300_sim.xacro"/>
-<xacro:include filename="$(find ds_sim)/urdf/nortek1000_sim.xacro"/>
-<xacro:include filename="$(find ds_sim)/urdf/xeos_gps_sim.xacro"/>
-<xacro:include filename="$(find ds_sim)/urdf/avtrak_sim.xacro"/>
-<xacro:include filename="$(find ds_sim)/urdf/resonAUV3_sim.xacro"/>
-<xacro:include filename="$(find ds_sim)/urdf/norbitWBMS_bathy_sim.xacro"/>
-<xacro:include filename="$(find ds_sim)/urdf/norbitWBMS_3D_sim.xacro"/>
-<xacro:include filename="$(find ds_sim)/urdf/basic_camera_sim.xacro"/>
-<xacro:include filename="$(find ds_sim)/urdf/dspl_seasphere_sim.xacro"/>
+<xacro:macro name="norbitWBMS_3D_sim" params="name parent_link xyz rpy robot_namespace topic">
+  <gazebo reference="${name}_link">
+    <material>Gazebo/Black</material>
+  </gazebo>
+  <!-- Gazebo plugin to actually take measurements! -->
+    <gazebo reference="${parent_link}">
+        <sensor name="${name}_sensor" type="ray">
+            <always_on>1</always_on>
+            <pose frame="">${xyz} ${rpy}</pose>
+            <visualize>true</visualize>
+            <update_rate>5</update_rate>
+            <ray>
+                <!-- These are our beams.  They're limited equi-angular, but the distinction probably
+                     doesn't matter -->
+                <scan>
+                    <horizontal>
+                        <samples>512</samples>
+                        <resolution>0.40</resolution>
+                        <min_angle>-${pi/180*100}</min_angle>
+                        <max_angle>${pi/180*100}</max_angle>
+                    </horizontal>
+                </scan>
+                <range>
+                    <min>0.2</min>
+                    <max>275</max>
+                    <resolution>0.01</resolution>
+                </range>
+            </ray>
+            <plugin name="${name}_sensor_controller" filename="libgazebo_ros_laser.so">
+                <topicName>topic</topicName>
+                <frameName>${name}_link</frameName>
+            </plugin>
+    </sensor>
+  </gazebo>
+</xacro:macro>
 </robot>

File: urdf/norbitWBMS_bathy_sim.xacro (robot description, xacro)
@@ -1,5 +1,5 @@
 <?xml version="1.0"?>
 <!--
-Copyright 2018 Woods Hole Oceanographic Institution
+Copyright 2019 Woods Hole Oceanographic Institution
 Redistribution and use in source and binary forms, with or without
 modification, are permitted provided that the following conditions are met:
@@ -25,14 +25,38 @@
 -->
 <robot xmlns:xacro="http://www.ros.org/wiki/xacro">
-<xacro:include filename="$(find ds_sim)/urdf/phins_sim.xacro"/>
-<xacro:include filename="$(find ds_sim)/urdf/paro_sim.xacro"/>
-<xacro:include filename="$(find ds_sim)/urdf/rdi300_sim.xacro"/>
-<xacro:include filename="$(find ds_sim)/urdf/nortek1000_sim.xacro"/>
-<xacro:include filename="$(find ds_sim)/urdf/xeos_gps_sim.xacro"/>
-<xacro:include filename="$(find ds_sim)/urdf/avtrak_sim.xacro"/>
-<xacro:include filename="$(find ds_sim)/urdf/resonAUV3_sim.xacro"/>
-<xacro:include filename="$(find ds_sim)/urdf/norbitWBMS_bathy_sim.xacro"/>
-<xacro:include filename="$(find ds_sim)/urdf/norbitWBMS_3D_sim.xacro"/>
-<xacro:include filename="$(find ds_sim)/urdf/basic_camera_sim.xacro"/>
-<xacro:include filename="$(find ds_sim)/urdf/dspl_seasphere_sim.xacro"/>
+<xacro:macro name="norbitWBMS_bathy_sim" params="name parent_link xyz rpy topic">
+  <gazebo reference="${name}_link">
+    <material>Gazebo/Black</material>
+  </gazebo>
+  <!-- Gazebo plugin to actually take measurements! -->
+    <gazebo reference="${parent_link}">
+        <sensor name="${name}_sensor" type="ray">
+            <always_on>1</always_on>
+            <pose frame="">${xyz} ${rpy}</pose>
+            <visualize>true</visualize>
+            <update_rate>5</update_rate>
+            <ray>
+                <!-- These are our beams.  They're limited equi-angular, but the distinction probably
+                     doesn't matter -->
+                <scan>
+                    <horizontal>
+                        <samples>512</samples>
+                        <resolution>0.40</resolution>
+                        <min_angle>-${pi/180*100}</min_angle>
+                        <max_angle>${pi/180*100}</max_angle>
+                    </horizontal>
+                </scan>
+                <range>
+                    <min>0.2</min>
+                    <max>275</max>
+                    <resolution>0.01</resolution>
+                </range>
+            </ray>
+            <plugin name="${name}_sensor_controller" filename="libgazebo_ros_laser.so">
+                <topicName>${topic}</topicName>
+                <frameName>${name}_link</frameName>
+            </plugin>
+    </sensor>
+  </gazebo>
+</xacro:macro>
 </robot>

File: urdf/nortek1000_sim.xacro (robot description, xacro)
@@ -25,5 +25,5 @@
 -->
 <robot xmlns:xacro="http://www.ros.org/wiki/xacro">
-<xacro:macro name="rdi_workhorse_300_sim" params="name parent_link xyz rpy robot_namespace dvl_topic ranges_topic">
+<xacro:macro name="nortek1000_sim" params="name parent_link xyz rpy robot_namespace dvl_topic ranges_topic">
   <gazebo reference="${name}_link">
     <material>Gazebo/Green</material>
@@ -32,20 +32,8 @@
     <sensor name="${name}_sensor" type="dsros_dvl">
       <always_on>1</always_on>
-      <update_rate>2.0</update_rate>
+      <update_rate>5.0</update_rate>
       <pose frame="">${xyz} ${rpy}</pose>
       <!-- This plugin MUST be included, because SDF sucks -->
       <plugin name="${name}_sensor_controller" filename="libdsros_ros_dvl.so">
-        <!--  300kHz DVL -->
-        <minRange>1.0</minRange>
-        <maxRange>200</maxRange>
-        <maxRangeDiff>10</maxRangeDiff>
-        <beamAngleDeg>30.0</beamAngleDeg>
-        <beamWidthDeg>4.0</beamWidthDeg>
-        <beamAzimuthDeg1>180</beamAzimuthDeg1>
-        <beamAzimuthDeg2>0</beamAzimuthDeg2>
-        <beamAzimuthDeg3>90</beamAzimuthDeg3>
-        <beamAzimuthDeg4>-90</beamAzimuthDeg4>
-        <pos_z_down>false</pos_z_down>
-        <collide_bitmask>0x0001</collide_bitmask>
         <robotNamespace>${robot_namespace}</robotNamespace>
         <topicName>${dvl_topic}</topicName>
@@ -53,5 +41,5 @@
         <frameName>${name}_link</frameName>
         <pointcloudFrame>${parent_link}</pointcloudFrame>
-        <updateRateHZ>2.0</updateRateHZ>
+        <updateRateHZ>5.0</updateRateHZ>
         <!--
         <gaussianNoiseBeamVel>0.01</gaussianNoiseBeamVel>
@@ -60,23 +48,19 @@
         <gaussianNoiseBeamVel>0.00</gaussianNoiseBeamVel>
         <gaussianNoiseBeamRange>0.0</gaussianNoiseBeamRange>
+        <!--  1000MHz DVL -->
+        <minRange>0.22</minRange>
+        <maxRange>55.16</maxRange>
+        <maxRangeDiff>10</maxRangeDiff>
+        <beamAngleDeg>25.0</beamAngleDeg>
+        <beamWidthDeg>4.0</beamWidthDeg>
+        <beamAzimuthDeg1>-135</beamAzimuthDeg1>
+        <beamAzimuthDeg2>135</beamAzimuthDeg2>
+        <beamAzimuthDeg3>45</beamAzimuthDeg3>
+        <beamAzimuthDeg4>-45</beamAzimuthDeg4>
+        <pos_z_down>true</pos_z_down>
+        <collide_bitmask>0x0001</collide_bitmask>
       </plugin>
     </sensor>
   </gazebo>
-        <!--  600kHz DVL -->
-        <!--
-        <minRange>0.7</minRange>
-        <maxRange>90</maxRange>
-        <maxRangeDiff>10</maxRangeDiff>
-        <beamAngleDeg>30.0</beamAngleDeg>
-        <beamWidthDeg>2.0</beamWidthDeg>
-        -->
-        <!-- 1200kHz DVL -->
-        <!--
-        <minRange>0.5</minRange>
-        <maxRange>45</maxRange>
-        <maxRangeDiff>10</maxRangeDiff>
-        <beamAngleDeg>30.0</beamAngleDeg>
-        <beamWidthDeg>1.5</beamWidthDeg>
-        -->
 </xacro:macro>
 </robot>
