Commit message: Getting sim ready for njr sim

File: urdf/paro_sim.xacro (robot description, xacro)
@@ -37,5 +37,5 @@
           <robotNamespace>${robot_namespace}</robotNamespace>
           <topicName>${topic}</topicName>
-          <frameName>world</frameName>
+          <frameName>${name}_link</frameName>
           <updateRateHZ>5</updateRateHZ>
           <!-- Actually in decibars, but pretty close to meters -->

File: urdf/phins_sim.xacro (robot description, xacro)
@@ -25,5 +25,5 @@
 -->
 <robot xmlns:xacro="http://www.ros.org/wiki/xacro">
-<xacro:macro name="phins_sim" params="name parent_link xyz rpy robot_namespace ins_topic gyro_topic att_topic">
+<xacro:macro name="phins_sim" params="name parent_link xyz rpy robot_namespace ins_topic gyro_topic att_topic phinsbin_topic">
   <gazebo reference="${name}_link">
     <material>Gazebo/Grey</material>
@@ -32,5 +32,5 @@
     <sensor name="${name}_sensor" type="dsros_ins">
       <always_on>1</always_on>
-      <update_rate>10.000</update_rate>
+      <update_rate>100.000</update_rate>
       <pose frame="">${xyz} ${rpy}</pose>
       <plugin name="${name}_sensor_controller" filename="libdsros_ros_ins.so">
@@ -39,6 +39,8 @@
         <gyroTopicName>${gyro_topic}</gyroTopicName>
         <attTopicName>${att_topic}</attTopicName>
-        <frameName>world</frameName>
+        <phinsbinTopicName>${phinsbin_topic}</phinsbinTopicName>
+        <frameName>${name}_link</frameName>
         <updateRateHZ>10</updateRateHZ>
+        <phinsbinUpdateRateHZ>100</phinsbinUpdateRateHZ>
         <gaussianNoisePR>0.001</gaussianNoisePR>
         <gaussianNoiseY>0.01</gaussianNoiseY>
