Commit message: Added option to turn off high-rate phinsbin messages, shiny new Reson plugin

File: urdf/norbitWBMS_bathy_sim.xacro (robot description, xacro)
@@ -25,5 +25,5 @@
 -->
 <robot xmlns:xacro="http://www.ros.org/wiki/xacro">
-<xacro:macro name="norbitWBMS_bathy_sim" params="name parent_link xyz rpy topic">
+<xacro:macro name="norbitWBMS_bathy_sim" params="name parent_link xyz rpy robot_namespace topic">
   <gazebo reference="${name}_link">
     <material>Gazebo/Black</material>
@@ -53,7 +53,16 @@
                 </range>
             </ray>
+            <!--
             <plugin name="${name}_sensor_controller" filename="libgazebo_ros_laser.so">
                 <topicName>${topic}</topicName>
                 <frameName>${name}_link</frameName>
+            </plugin>
+            -->
+            <plugin name="${name}_sensor_controller" filename="libdsros_ros_reson.so">
+                <robotNamespace>${robot_namespace}</robotNamespace>
+                <topicName>${topic}</topicName>
+                <frameName>${name}_link</frameName>
+                <updateRateHZ>5.0</updateRateHZ>
+                <gaussianNoise>0.0</gaussianNoise>
             </plugin>
     </sensor>
